File: pcb/promicro_holder.kicad_pcb (KiCad board)
At the start: 2 copper layers, 36.3 x 31.1 mm, 11 parts, among them J1 MJ-4PP-9, J3 Conn_01x08, J4 Conn_01x08, J6 MJ-4PP-9, U1 ProMicro

Commit message: second commit
Routing:
- net dummydata: track 50.9 -> 52.9 mm
