File: pcb/promicro_holder.sch (KiCad schematic (older format))
At the start: 5 parts, among them J1 MJ-4PP-9, J3 Conn_01x08, J4 Conn_01x08, J6 MJ-4PP-9, U1 ProMicro

Commit message: update
Parts:
- J3, J4: symbol Connector_Generic:Conn_01x08 -> promicro_holder-rescue:Conn_01x08-Connector_Generic
Changed lines of the file:
@@
 encoding utf-8
 Sheet 1 1
-Title "SU120 Yakitori Keyboard"
+Title "pro micro holder"
 Date ""
-Rev "8"
-Comp "@e3w2q"
+Rev "3"
+Comp "ergohaven"
 Comment1 ""
 Comment2 ""
@@
 Y5
 $Comp
-L power:GND #PWR0101
+L promicro_holder-rescue:GND-power #PWR0101
 U 1 1 5CE3BEE4
 P 1050 950
@@
 $EndComp
 $Comp
-L power:PWR_FLAG #FLG0101
+L promicro_holder-rescue:PWR_FLAG-power #FLG0101
 U 1 1 5CE3BEEA
 P 1050 800
@@
 $EndComp
 $Comp
-L power:PWR_FLAG #FLG0102
+L promicro_holder-rescue:PWR_FLAG-power #FLG0102
 U 1 1 5CE3BEF0
 P 700 950
@@
 	700  800  700  950
 $Comp
-L power:VCC #PWR0102
+L promicro_holder-rescue:VCC-power #PWR0102
 U 1 1 5CE3E880
 P 700 800
@@
 $EndComp
 $Comp
-L power:VCC #PWR0103
+L promicro_holder-rescue:VCC-power #PWR0103
 U 1 1 5CE3F20D
 P 5000 1150
@@
 $EndComp
 $Comp
-L power:GND #PWR0104
+L promicro_holder-rescue:GND-power #PWR0104
 U 1 1 5CE4B3AC
 P 4650 2600
@@
 data
 $Comp
-L power:GND #PWR0109
+L promicro_holder-rescue:GND-power #PWR0109
 U 1 1 5CE6AB53
 P 1550 4450
@@
 $EndComp
 $Comp
-L power:VCC #PWR0110
+L promicro_holder-rescue:VCC-power #PWR0110
 U 1 1 5CE6AC90
 P 1550 4050
@@
 NoConn ~ 1250 4100
 $Comp
-L Connector_Generic:Conn_01x08 J3
+L promicro_holder-rescue:Conn_01x08-Connector_Generic J3
 U 1 1 5CE5F218
 P 3900 3250
@@
 $EndComp
 $Comp
-L Connector_Generic:Conn_01x08 J4
+L promicro_holder-rescue:Conn_01x08-Connector_Generic J4
 U 1 1 5CE5F3DE
 P 1750 3250
@@
 dummyGND
 $Comp
-L power:GND #PWR01
+L promicro_holder-rescue:GND-power #PWR01
 U 1 1 5CF6A65C
 P 4300 2600
